File: ai03-macropad-pcb.sch (KiCad schematic (older format))
At the start: 74 parts, among them J1 Conn_01x06, SW1 SW_Push, U1 ATmega32U4-MU, Y1 16Mhz

Commit message: RevA Routing complete
Parts:
- added D25: LED, LED_SMD:LED_0603_1608Metric, symbol Device:LED
- added R9: 1k, Resistor_SMD:R_0603_1608Metric, symbol Device:R_Small
- H1, H2, H3, H4: footprint MountingHole:MountingHole_3.2mm_M3_Pad_TopBottom -> MountingHole:MountingHole_3.2mm_M3_DIN965_Pad
- SW1: footprint random-keyboard-parts:SKQG-1155865 -> Button_Switch_SMD:SW_SPST_CK_KXT3
Connections:
- net +5V: now also D14.4 (VCC), J1.6 (Pin_6)
- net COL0: now also U1.40 (PF1); no longer U1.41 (PF0)
- net D+: no longer R5.1, U1.4 (D+)
- net D-: no longer R6.1, U1.3 (D-)
- net GND: now also R9.1; no longer C14.2
- net RGB1: now also D21.4 (DIN); no longer D11.4 (DIN)
- net VCC: no longer D14.4 (VCC), J1.6 (Pin_6)
- net at U1.37 (PF6): now also D25.2 (A)
- net at R8.2: now also U1.41 (PF0); no longer U1.40 (PF1)
- net D12: now reaches D12.4 (DIN)
- net D12: now also D22.2 (DOUT); no longer D18.2 (DOUT)
- net D13: now reaches D13.4 (DIN)
- net D13: now also D24.2 (DOUT); no longer D19.2 (DOUT)
- net D11: now reaches D21.2 (DOUT)
- net D11: now also D11.4 (DIN); no longer D22.4 (DIN)
- net D23: now reaches D23.4 (DIN)
- net D23: now also D20.2 (DOUT); no longer D24.2 (DOUT)
- net D24: now reaches D24.4 (DIN)
- net D24: now also D19.2 (DOUT); no longer D22.2 (DOUT)
- net at R3.2, SW1.1: now also C14.2
- removed net RGB2: D20.2 (DOUT), D21.4 (DIN)
- new net: R6.1, U1.3 (D-)
- new net: R5.1, U1.4 (D+)
- new net: D25.1 (K), R9.2
- new net D22: D18.2 (DOUT), D22.4 (DIN)
- no-connect marks 3 -> 18
Other:
- moved on the sheet: R3, R5, R6, R8

Commit message: RevA DRC check
Connections:
- net D_N: now reaches R6.1, U1.3 (D-)
- net D_P: now reaches R5.1, U1.4 (D+)
Other:
- moved on the sheet: R5, R6
Changed lines of the file:
@@
 L Device:R_Small R6
 U 1 1 6073035A
-P 8450 3800
-F 0 "R6" V 8550 3800 50  0000 C BNN
-F 1 "22" V 8450 3800 39  0000 C CNN
-F 2 "Resistor_SMD:R_0603_1608Metric" H 8450 3800 50  0001 C CNN
-F 3 "~" H 8450 3800 50  0001 C CNN
-	1    8450 3800
+P 8200 3800
+F 0 "R6" V 8300 3800 50  0000 C BNN
+F 1 "22" V 8200 3800 39  0000 C CNN
+F 2 "Resistor_SMD:R_0603_1608Metric" H 8200 3800 50  0001 C CNN
+F 3 "~" H 8200 3800 50  0001 C CNN
+	1    8200 3800
 	0    1    1    0
 $EndComp
@@
 L Device:R_Small R5
 U 1 1 6072EE07
-P 8450 3700
-F 0 "R5" V 8350 3700 50  0000 C TNN
-F 1 "22" V 8450 3700 39  0000 C CNN
-F 2 "Resistor_SMD:R_0603_1608Metric" H 8450 3700 50  0001 C CNN
-F 3 "~" H 8450 3700 50  0001 C CNN
-	1    8450 3700
+P 8200 3700
+F 0 "R5" V 8100 3700 50  0000 C TNN
+F 1 "22" V 8200 3700 39  0000 C CNN
+F 2 "Resistor_SMD:R_0603_1608Metric" H 8200 3700 50  0001 C CNN
+F 3 "~" H 8200 3700 50  0001 C CNN
+	1    8200 3700
 	0    1    1    0
 $EndComp
@@
 	5250 7200 5250 7250
 Wire Wire Line
-	8150 3800 8350 3800
-Wire Wire Line
-	8150 3700 8350 3700
-Wire Wire Line
-	8900 3800 8550 3800
-Wire Wire Line
-	8550 3700 8900 3700
-Text GLabel 8150 3800 0    50   Input ~ 0
+	7900 3800 8100 3800
+Wire Wire Line
+	7900 3700 8100 3700
+Text GLabel 7900 3800 0    50   Input ~ 0
 D-
-Text GLabel 8150 3700 0    50   Input ~ 0
+Text GLabel 7900 3700 0    50   Input ~ 0
 D+
 $Comp
@@
 NoConn ~ 10100 2700
 NoConn ~ 10100 5600
+Wire Wire Line
+	8300 3700 8400 3700
+Wire Wire Line
+	8300 3800 8400 3800
+Wire Wire Line
+	8900 3700 8800 3700
+Wire Wire Line
+	8900 3800 8800 3800
+Text GLabel 8800 3800 0    50   Input ~ 0
+D_N
+Text GLabel 8400 3800 2    50   Output ~ 0
+D_N
+Text GLabel 8400 3700 2    50   Output ~ 0
+D_P
+Text GLabel 8800 3700 0    50   Input ~ 0
+D_P
 $EndSCHEMATC
