File: ai03-macropad-pcb.sch (KiCad schematic (older format))
At the start: 76 parts, among them J1 Conn_01x06, SW1 SW_Push, U1 ATmega32U4-MU, Y1 16Mhz

Commit message: Gerbers pre-prod
Parts:
- D4: value D_Schottky_Small -> 450mV @ 500mA
Changed lines of the file:
@@
 P 1900 1650
 F 0 "D4" H 1900 1550 50  0000 C CNN
-F 1 "D_Schottky_Small" H 1900 1750 50  0000 C CNN
+F 1 "450mV @ 500mA" H 1900 1750 50  0000 C CNN
 F 2 "Diode_SMD:D_SOD-123" V 1900 1650 50  0001 C CNN
 F 3 "~" V 1900 1650 50  0001 C CNN
